File: 0.5u Headphone:line out/0.5u Headphone:line out-rounded.kicad_pcb (KiCad board)
At the start: 2 copper layers, 86.4 x 30.5 mm, 58 parts, among them J1 IN L, J2 IN R, J3 Eurorack_Power_10pin_Unshroud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, J4 3.5mm_Stereo, J5 Conn_02x03, J6 Conn_01x04_Pin, Q1 3904, Q2 3904, U1 TL074, U3 NE5532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

Commit message: Min Max Switch
Other:
- board text added: "Red"
