File: 0.5u Line in/0.5u Line in.kicad_pcb (KiCad board)
At the start: 2 copper layers, 86.4 x 30.5 mm, 40 parts, among them J1 Eurorack_Power_10pin_Unshroud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, J2 Conn_01x04_Pin, J3 Conn_02x03, J4 IN R, J5 IN R, Q1 3904, Q2 3904, U1 TL074

Commit message: Min Max Switch
Parts:
- moved J1 10.5 mm to (182.2, 49.5), turned to -90 degrees
- moved D4 0.06 mm to (183.6, 33.0)
- moved Q2 0.06 mm to (177.9, 33.0)
- moved R13 0.06 mm to (188.7, 33.3)
- moved R14 0.06 mm to (186.2, 33.3)
Routing:
- net Out R: track 80.9 -> 81.4 mm
