File: 0.5u Line in/0.5u Line in.kicad_sch (KiCad schematic)
At the start: 36 parts, among them J1 Eurorack_Power_10pin_Unshroud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, J3 Conn_02x03, J4 IN R, J5 Conn_01x04_Pin, J5 IN R, Q1 3904, Q2 3904, U1 TL074

Commit message: Min Max Switch
Parts:
- J4: value IN R -> IN L
- RV1, RV2: value R_Potentiometer -> A10k
Changed lines of the file:
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@@
       (effects (font (size 1.27 1.27)))
     )
-    (property "Value" "R_Potentiometer" (at 104.14 96.52 90)
+    (property "Value" "A10k" (at 104.14 96.52 90)
       (effects (font (size 1.27 1.27)))
     )
@@
       (effects (font (size 1.27 1.27)))
     )
-    (property "Value" "R_Potentiometer" (at 104.14 44.45 90)
+    (property "Value" "A10k" (at 104.14 44.45 90)
       (effects (font (size 1.27 1.27)))
     )
@@
       (effects (font (size 1.524 1.524)))
     )
-    (property "Value" "IN R" (at 187.96 49.53 0)
+    (property "Value" "IN L" (at 187.96 49.53 0)
       (effects (font (size 1.524 1.524)))
     )
